File: KiCAD/(N)AND/(N)AND.kicad_pcb (KiCad board)
At the start: 2 copper layers, 71.1 x 62.2 mm, 18 parts, among them J1 Conn_01x02_Pin, J2 Conn_01x02_Pin, J3 Conn_01x02_Pin, J4 Conn_01x02_Pin, Q13 2N7000, Q14 2N7000, Q15 2N7000, Q3 2N7000, Q4 2N7000, Q5 2N7000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

Commit message: Cleanup
Parts:
- moved A1 14.5 mm to (234.2, 95.1)
- moved J1 14.5 mm to (202.4, 95.1)
- moved J2 14.5 mm to (202.4, 148.5)
- moved Q13 14.5 mm to (234.3, 112.9)
- moved Q4 14.5 mm to (250.7, 116.7)
- moved R15 14.5 mm to (208.8, 116.7)
- moved R5 14.5 mm to (203.7, 116.7)
- moved B1 14.5 mm to (249.4, 95.1)
- moved J4 14.5 mm to (260.9, 95.1)
- moved Q14 14.5 mm to (249.6, 112.9)
- moved Q15 14.5 mm to (226.7, 134.5)
- moved Q3 14.5 mm to (235.5, 116.7)
- moved Q5 14.5 mm to (227.8, 138.3)
- moved R16 14.5 mm to (208.8, 138.3)
- moved R6 14.5 mm to (203.7, 138.3)
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Routing:
- net (no net): track 56.6 -> 48.6 mm
- net GNDREF: track 79.6 -> 78.3 mm
- net VDD: vias 8 -> 6
Other:
- board text added: "&"
- board text added: "+V opens the Gate"
- board text added: "DRAIN"
- board text added: "Drains power from +V"
- board text added: "GATE"
- board text added: "MOSFET"
- board text added: "N-Channel"
- board text added: "N-Channel MOSFET :"
- board text added: "Provides a power Source"
- board text added: "SOURCE"
- board text added: "~{&}"
