File: KiCAD/NAND/NAND.kicad_pcb (KiCad board)
At the start: 2 copper layers, 58.4 x 40.6 mm, 13 parts, among them J1 Conn_01x02_Pin, J2 Conn_01x02_Pin, J3 Conn_01x02_Pin, J4 Conn_01x02_Pin, Q13 2N7000, Q14 2N7000, Q3 2N7000, Q4 2N7000, Y1 Conn_01x01_Pin

Commit message: Cleanup
Other:
- board text added: "~{&}"
Changed lines of the file:
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@@
+		)
+	)
+	(gr_text "~{&}"
+		(at 234.060295 116.687013 0)
+		(layer "F.Cu")
+		(effects
+			(font
+				(size 1.27 1.27)
+				(thickness 0.254)
+				(bold yes)
+			)
+			(justify left bottom)
+		)
+	)
+	(gr_text "~{&}"
+		(at 235.891332 116.679112 0)
+		(layer "B.Cu")
+		(effects
+			(font
+				(size 1.27 1.27)
+				(thickness 0.254)
+				(bold yes)
+			)
+			(justify left bottom mirror)
 		)
 	)
