File: KiCAD/XOR_LED/XOR_LED.kicad_pcb (KiCad board)
At the start: 2 copper layers, 104.1 x 119.4 mm, 44 parts, among them J1 Conn_01x02_Pin, J2 Conn_01x02_Pin, J3 Conn_01x02_Pin, J4 Conn_01x02_Pin, Q1 2N7000, Q11 2N7000, Q12 2N7000, Q13 2N7000, Q14 2N7000, Q15 2N7000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

Commit message: Cleanup
Parts:
- moved J1 3.22 mm to (52.1, 43.2), turned to -90 degrees
- moved J4 1.49 mm to (146.1, 43.2), turned to -90 degrees
- moved J3 1.48 mm to (146.1, 154.9), turned to -90 degrees
- moved J2 1.16 mm to (52.1, 154.9), turned to -90 degrees
Routing:
- net VDD: track 557.6 -> 560.8 mm
- net GNDREF: track 94.5 -> 93.9 mm
- net (no net): vias 0 -> 1
Other:
- board text added: "^"
- board text added: "~{^}"
