File: KiCAD/(N)OR/(N)OR.kicad_pcb (KiCad board)
At the start: 2 copper layers, 71.1 x 62.2 mm, 18 parts, among them J1 Conn_01x02_Pin, J2 Conn_01x02_Pin, J3 Conn_01x02_Pin, J4 Conn_01x02_Pin, Q13 2N7000, Q14 2N7000, Q15 2N7000, Q3 2N7000, Q4 2N7000, Q5 2N7000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

Commit message: (N)OR
Parts:
- moved Q3 15.1 mm to (234.9, 101.6)
- moved Q13 15.1 mm to (233.8, 97.8)
- moved A1 13.8 mm to (233.7, 81.3)
- moved B1 13.8 mm to (248.9, 81.3)
- moved J4 13.8 mm to (260.3, 81.3)
- moved J1 13.8 mm to (201.9, 81.3)
- moved R15 7.47 mm to (208.3, 109.3)
- moved R5 7.47 mm to (203.2, 109.3)
- moved J2 0.54 mm to (201.9, 148.6)
- moved J3 0.54 mm to (260.3, 148.6)
- moved Q15 0.54 mm to (226.2, 134.7)
- moved Q5 0.54 mm to (227.3, 138.5)
- moved R16 0.54 mm to (208.3, 138.5)
- moved R6 0.54 mm to (203.2, 138.5)
- moved Y2 0.54 mm to (242.6, 148.6)
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Connections:
- Q13 pad 1: Net-(Q13-S) -> GNDREF
- Q14 pad 3: Net-(Q13-S) -> Net-(Q13-D)
- Q3 pad 1: Net-(Q13-S) -> GNDREF
- Q4 pad 3: Net-(Q13-S) -> Net-(Q13-D)
Routing:
- net GNDREF: track 78.3 -> 133.1 mm, vias 5 -> 2
- net Net-(Q13-D): track 89.3 -> 142.9 mm
- net VDD: track 263.6 -> 287.1 mm, vias 6 -> 5
- net Net-(Q13-S): track 19.6 -> 0.00 mm
- net Net-(B1-Pin_1): track 24.4 -> 36.7 mm, vias 0 -> 2
- net (no net): track 48.6 -> 38.9 mm
- net Net-(A1-Pin_1): track 27.9 -> 25.1 mm
Other:
- board size 71.1 x 62.2 mm -> 69.8 x 74.9 mm
- board text added: "1st Digit"
- board text added: "2nd Digit"
- board text added: "A | B"
- board text added: "Number"
- board text added: "OR"
- board text added: "Resistor Colour Code"
- board text added: "of 0's"
- board text added: "~{A | B}"
- board text removed: "&"
- board text removed: "+V Opens the Gate"
- board text removed: "A & B"
- board text removed: "AND"
- board text removed: "DRAIN"
- board text removed: "Drains power from +V"
- board text removed: "GATE"
- board text removed: "MOSFET"
- board text removed: "N-Channel"
- board text removed: "N-Channel MOSFET :"
- board text removed: "Provides a power Source"
- board text removed: "SOURCE"
- board text removed: "~{&}"
- board text removed: "~{A & B}"

Commit message: (N)OR_LED
Changed lines of the file:
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@@
 	)
 	(gr_line
-		(start 220.559532 148.450247)
-		(end 219.581492 148.450247)
-		(stroke
-			(width 0.254)
-			(type default)
-		)
-		(layer "B.Cu")
-	)
-	(gr_line
-		(start 225.80226 150.109704)
-		(end 225.802462 150.10823)
+		(start 245.913712 148.462954)
+		(end 244.935672 148.462954)
 		(stroke
 			(width 0.254)
@@
 	)
 	(gr_line
-		(start 250.828379 150.098095)
-		(end 250.828581 150.096621)
+		(start 225.564339 150.087545)
+		(end 225.564541 150.086071)
 		(stroke
 			(width 0.254)
@@
 	)
 	(gr_arc
-		(start 225.80226 150.109704)
-		(mid 223.573792 149.729065)
-		(end 221.710033 148.449471)
+		(start 251.15644 150.122411)
+		(mid 248.927972 149.741772)
+		(end 247.064213 148.462178)
 		(stroke
 			(width 0.254)
@@
 	)
 	(gr_line
-		(start 225.336465 147.714569)
-		(end 227.093686 147.714569)
+		(start 250.690645 147.727276)
+		(end 252.447866 147.727276)
 		(stroke
 			(width 0.254)
@@
 	)
 	(gr_line
-		(start 246.740211 148.438638)
-		(end 246.736152 148.437862)
+		(start 221.476171 148.428088)
+		(end 221.472112 148.427312)
 		(stroke
 			(width 0.254)
@@
 	)
 	(gr_arc
-		(start 246.740211 148.438638)
-		(mid 248.612515 147.114461)
-		(end 250.870543 146.714066)
+		(start 221.476171 148.428088)
+		(mid 223.348482 147.103924)
+		(end 225.606503 146.703516)
 		(stroke
 			(width 0.254)
@@
 	)
 	(gr_arc
-		(start 250.828379 150.098095)
-		(mid 248.599909 149.71746)
-		(end 246.736152 148.437862)
+		(start 225.564339 150.087545)
+		(mid 223.335869 149.70691)
+		(end 221.472112 148.427312)
 		(stroke
 			(width 0.254)
@@
 	)
 	(gr_arc
-		(start 250.828581 150.096621)
-		(mid 250.204203 148.396993)
-		(end 250.870949 146.713526)
+		(start 225.564541 150.086071)
+		(mid 224.940163 148.386443)
+		(end 225.606909 146.702976)
 		(stroke
 			(width 0.254)
@@
 		(layer "B.Cu")
 	)
-	(gr_line
-		(start 221.714092 148.450247)
-		(end 221.710033 148.449471)
-		(stroke
-			(width 0.254)
-			(type default)
-		)
-		(layer "B.Cu")
-	)
 	(gr_arc
 		(start 218.566705 82.1447)
@@
 	)
 	(gr_line
-		(start 225.84483 146.725135)
-		(end 225.844424 146.725675)
-		(stroke
-			(width 0.254)
-			(type default)
-		)
-		(layer "B.Cu")
-	)
-	(gr_line
-		(start 250.362584 149.312109)
-		(end 252.119805 149.312109)
+		(start 225.098544 149.301559)
+		(end 226.855765 149.301559)
 		(stroke
 			(width 0.254)
@@
 	)
 	(gr_circle
-		(center 221.079092 148.450247)
-		(end 221.079092 148.958247)
+		(center 246.433272 148.462954)
+		(end 246.433272 148.970954)
 		(stroke
 			(width 0.254)
@@
 	)
 	(gr_arc
-		(start 225.802462 150.10823)
-		(mid 225.178075 148.408598)
-		(end 225.84483 146.725135)
+		(start 251.156642 150.120937)
+		(mid 250.532255 148.421305)
+		(end 251.19901 146.737842)
 		(stroke
 			(width 0.254)
@@
 	)
 	(gr_line
-		(start 225.336465 149.323718)
-		(end 227.093686 149.323718)
+		(start 250.690645 149.336425)
+		(end 252.447866 149.336425)
 		(stroke
 			(width 0.254)
@@
 	)
 	(gr_line
-		(start 250.362584 147.70296)
-		(end 252.119805 147.70296)
+		(start 225.098544 147.69241)
+		(end 226.855765 147.69241)
 		(stroke
 			(width 0.254)
@@
 	)
 	(gr_arc
-		(start 221.714092 148.450247)
-		(mid 223.586392 147.126048)
-		(end 225.844424 146.725675)
+		(start 247.068272 148.462954)
+		(mid 248.940572 147.138755)
+		(end 251.198604 146.738382)
 		(stroke
 			(width 0.254)
@@
 	)
 	(gr_line
-		(start 250.870949 146.713526)
-		(end 250.870543 146.714066)
+		(start 225.606909 146.702976)
+		(end 225.606503 146.703516)
 		(stroke
 			(width 0.254)
@@
 	)
 	(gr_line
-		(start 246.736152 148.438638)
-		(end 244.607611 148.438638)
+		(start 221.472112 148.428088)
+		(end 219.343571 148.428088)
 		(stroke
 			(width 0.254)
@@
 	)
 	(segment
-		(start 249.073767 148.199204)
-		(end 249.073767 149.215204)
+		(start 223.747947 147.907069)
+		(end 223.747947 148.923069)
 		(width 0.2)
 		(layer "B.Cu")
@@
 	)
 	(segment
-		(start 223.920978 147.857023)
-		(end 223.920978 148.873023)
+		(start 249.314826 148.097008)
+		(end 249.314826 149.113008)
 		(width 0.2)
 		(layer "B.Cu")
@@
 	)
 	(segment
+		(start 248.804011 147.70315)
+		(end 249.820011 147.70315)
+		(width 0.2)
+		(layer "B.Cu")
+		(net 0)
+	)
+	(segment
 		(start 210.057705 82.8675)
 		(end 210.184705 82.9945)
@@
 	)
 	(segment
-		(start 248.565767 147.691204)
-		(end 249.581767 147.691204)
-		(width 0.2)
-		(layer "B.Cu")
-		(net 0)
-	)
-	(segment
 		(start 208.787435 80.074367)
 		(end 208.914435 79.947367)
@@
 	)
 	(group ""
-		(members "164f51fc-f3f7-4605-be37-ec8e66ed987b" "1d56fd1a-1012-4e93-8268-17ccba472532"
-			"30713374-0b52-48fc-a5db-3fe2c268d55a" "36b03394-5b95-4935-bb69-f11caea5e578"
-			"5cb2dd8d-6110-49ce-a069-7c7d0410a3f1" "6e8ea84e-342e-4671-bf2b-0ef8fa9dceaa"
-			"91c20777-1875-4897-86e1-a7be037447b4" "9893b303-c74e-4eac-b301-79ac359c8e78"
-			"a43ae842-8973-4582-896d-f25ca72afdb1" "cf560a8c-a7ea-47ca-beae-f3de367cb094"
+		(members "164f51fc-f3f7-4605-be37-ec8e66ed987b" "30713374-0b52-48fc-a5db-3fe2c268d55a"
+			"36b03394-5b95-4935-bb69-f11caea5e578" "91c20777-1875-4897-86e1-a7be037447b4"
+			"9893b303-c74e-4eac-b301-79ac359c8e78" "a43ae842-8973-4582-896d-f25ca72afdb1"
+			"a69742f3-c06c-4f00-861a-f5f1920ef5d3" "cf560a8c-a7ea-47ca-beae-f3de367cb094"
 			"f710f5ae-c3df-4acb-a6c2-379536766871"
 		)
 	)
 	(group ""
+		(members "22fcbaaf-1ff4-4eac-a8b4-46bb8d689ccf" "403dd6f9-19a1-4ff5-a5b3-2c2094659f67"
+			"40451896-61cf-41bc-90da-ce8f38a93de8" "4c0dcb25-4cf3-42e2-9384-6a19abf092e3"
+			"4ecc0d03-32da-4ecb-8330-936594110122" "4f9215e1-1c24-47e1-9e1a-335df6e4fe01"
+			"73955456-4a4e-4924-805b-e25abec4993e" "d0e33005-7604-4564-9c9e-059caf3a5be0"
+			"f94a83f3-256b-44ce-a5a0-db2adb4603f2" "fac428fa-60f9-4519-85d2-c4ad46d99769"
+		)
+	)
+	(group ""
 		(members "1374eeb0-28b8-43fa-af40-15bf90cf7120" "13ec4a57-3412-4ff0-b435-d4fe6040a8fb"
 			"22a31ac9-d40e-47cf-b336-19be7bd58066" "2b7d636b-f69f-45ef-be8b-8f00f156b025"
@@
 		)
 	)
-	(group ""
-		(members "22fcbaaf-1ff4-4eac-a8b4-46bb8d689ccf" "403dd6f9-19a1-4ff5-a5b3-2c2094659f67"
-			"40451896-61cf-41bc-90da-ce8f38a93de8" "4c0dcb25-4cf3-42e2-9384-6a19abf092e3"
-			"4ecc0d03-32da-4ecb-8330-936594110122" "4f9215e1-1c24-47e1-9e1a-335df6e4fe01"
-			"73955456-4a4e-4924-805b-e25abec4993e" "98a63ead-b11f-45ed-aa9c-6c1ec7ffe4e3"
-			"c97aff43-3c52-4d32-a164-63ff8ec11f2c" "d0e33005-7604-4564-9c9e-059caf3a5be0"
-			"f94a83f3-256b-44ce-a5a0-db2adb4603f2" "fac428fa-60f9-4519-85d2-c4ad46d99769"
-		)
-	)
