File: KiCAD/(N)OR_LED/(N)OR_LED.kicad_pcb (KiCad board)
At the start: 2 copper layers, 104.1 x 119.4 mm, 44 parts, among them J1 Conn_01x02_Pin, J2 Conn_01x02_Pin, J3 Conn_01x02_Pin, J4 Conn_01x02_Pin, Q1 2N7000, Q11 2N7000, Q12 2N7000, Q13 2N7000, Q14 2N7000, Q15 2N7000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

Commit message: (N)OR_LED
Parts:
- removed Q15, Q16: 2N7000, Package_TO_SOT_SMD:SOT-23
- removed Q5, Q6: 2N7000, Package_TO_SOT_THT:TO-92_Inline
- moved J1 135.3 mm to (186.7, 57.1)
- moved J2 135.1 mm to (186.7, 143.5)
- moved B1 130.3 mm to (237.5, 57.1)
- moved A1 130.3 mm to (217.2, 57.1)
- moved C1 129.9 mm to (226.1, 90.3)
- moved D2 129.9 mm to (237.5, 82.5)
- moved Q11 129.9 mm to (217.3, 68.6)
- moved Q4 129.9 mm to (236.2, 104.1)
- moved R11 129.9 mm to (191.8, 72.4)
- moved R14 129.9 mm to (247.5, 82.5)
- moved R15 129.9 mm to (191.8, 104.1)
- moved R3 129.9 mm to (201.9, 82.5)
- moved C2 129.9 mm to (227.3, 92.6)
- moved D1 129.9 mm to (217.2, 82.5)
- moved D11 129.9 mm to (218.4, 80.0)
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Routing:
- net Net-(A1-Pin_1): track 187.0 -> 20.2 mm, vias 2 -> 0
- net Net-(B1-Pin_1): track 151.5 -> 16.5 mm
- net VDD: track 560.8 -> 473.6 mm, vias 11 -> 10
- net GNDREF: track 93.9 -> 52.2 mm, vias 24 -> 3
- net (no net): track 0.00 -> 38.9 mm, vias 1 -> 0
- net Net-(Q13-D): track 175.3 -> 137.4 mm
- net Net-(Q15-S): track 19.7 -> 0.00 mm
Other:
- board size 104.1 x 119.4 mm -> 94 x 94 mm
- board text added: "( Y = A | B )"
- board text added: "(N)OR"
- board text added: "By putting capacitors around the board, we can ensure that clean power is always available where it will be required."
- board text added: "CERN-OSH-P-2.0"
- board text added: "In normal use of these demo boards, the capacitors will serve no useful function, and may be omitted!"
- board text added: "These {dblquote}batteries{dblquote} will help keep local power steady when other logic is causing power fluctuations. You could say it {dblquote}filters noise from the power{dblquote}."
- board text added: "Transistors require power to {dblquote}switch{dblquote}. One feature of a capacitor is to act like a tiny rechargeable battery."
- board text removed: "( Y = A ^ B )"
- board text removed: "(A | B) & A & B"
- board text removed: "A | B"
- board text removed: "Licence: CERN-OSH-P-2.0"
- board text removed: "OR"
- board text removed: "Transistors: N-Channel, Enhancement-Mode MOSFET (2N7000/2N7002 or equivalent)"
- board text removed: "X(N)OR"
