File: KiCAD/NOT/NOT.kicad_pcb (KiCad board)
At the start: 2 copper layers, 40.6 x 40.6 mm, 10 parts, among them J1 Conn_01x02_Pin, J2 Conn_01x02_Pin, J3 Conn_01x02_Pin, J4 Conn_01x02_Pin, Q13 2N7000, Q3 2N7000, Y1 Conn_01x01_Pin

Commit message: Cleanup
Other:
- board text added: "!"
Changed lines of the file:
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@@
 	)
 	(gr_line
-		(start 231.139705 129.54329)
+		(start 235.585 129.54329)
 		(end 228.591731 129.54329)
 		(stroke
@@
 		)
 	)
+	(gr_text "!"
+		(at 218.054688 115.814609 0)
+		(layer "F.Cu")
+		(effects
+			(font
+				(size 1.016 1.016)
+				(thickness 0.2032)
+				(bold yes)
+			)
+			(justify left bottom)
+		)
+	)
 	(gr_text "NOT"
 		(at 215.264705 107.95 0)
@@
 		)
 	)
+	(gr_text "!"
+		(at 218.171619 118.054278 0)
+		(layer "B.Cu")
+		(effects
+			(font
+				(size 1.016 1.016)
+				(thickness 0.2032)
+				(bold yes)
+			)
+			(justify left bottom)
+		)
+	)

Commit message: KiCAD: NOT_LED
Connections:
- Q13 pad 1: Net-(Q13-S) -> GNDREF
- Q3 pad 1: Net-(Q13-S) -> GNDREF
Routing:
- net GNDREF: track 33.0 -> 43.6 mm
- net Net-(Q13-S): track 2.95 -> 0.00 mm
Changed lines of the file:
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@@
 	(net 3 "VDD")
 	(net 4 "Net-(Q13-D)")
-	(net 5 "Net-(Q13-S)")
 	(footprint "Connector_PinHeader_2.54mm:PinHeader_1x01_P2.54mm_Vertical"
 		(layer "F.Cu")
@@
 			(layers "*.Cu" "*.Mask")
 			(remove_unused_layers no)
-			(net 5 "Net-(Q13-S)")
+			(net 2 "GNDREF")
 			(pinfunction "S")
 			(pintype "passive")
@@
 			)
 		)
+		(property ki_fp_filters "Connector*:*_1x??_*")
+		(sheetname "/")
+		(sheetfile "NOT.kicad_sch")
 		(attr through_hole)
 		(fp_line
@@
 			(layers "F.Cu" "F.Mask" "F.Paste")
 			(roundrect_rratio 0.25)
-			(net 5 "Net-(Q13-S)")
+			(net 2 "GNDREF")
 			(pinfunction "S")
 			(pintype "passive")
@@
 	)
 	(segment
+		(start 228.586283 129.561263)
+		(end 228.586283 126.922267)
+		(width 0.2)
+		(layer "F.Cu")
+		(net 2)
+	)
+	(segment
+		(start 236.219705 129.561263)
+		(end 228.586283 129.561263)
+		(width 0.4)
+		(layer "F.Cu")
+		(net 2)
+	)
+	(segment
+		(start 228.586283 126.922267)
+		(end 228.365279 126.701263)
+		(width 0.2)
+		(layer "F.Cu")
+		(net 2)
+	)
+	(segment
 		(start 236.219705 129.561263)
 		(end 236.219705 139.70329)
@@
 		(net 4)
 	)
-	(segment
-		(start 228.586283 129.561263)
-		(end 228.586283 126.922267)
-		(width 0.2)
-		(layer "F.Cu")
-		(net 5)
-	)
-	(segment
-		(start 228.586283 126.922267)
-		(end 228.365279 126.701263)
-		(width 0.2)
-		(layer "F.Cu")
-		(net 5)
-	)
 	(zone
