File: KiCAD/(N)AND_LED/(N)AND_LED.kicad_pcb (KiCad board)
At the start: 2 copper layers, 94 x 94 mm, 40 parts, among them J1 Conn_01x02_Pin, J2 Conn_01x02_Pin, J3 Conn_01x02_Pin, J4 Conn_01x02_Pin, Q1 2N7000, Q11 2N7000, Q12 2N7000, Q13 2N7000, Q14 2N7000, Q17 2N7000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

Commit message: KiCAD: (N)AND_LED
Parts:
- moved J3 16.5 mm to (270.5, 160.0)
- moved Y1 16.5 mm to (218.4, 160.0)
- moved ~{Y}1 16.5 mm to (245.1, 160.0)
- moved J2 16.4 mm to (186.7, 159.9)
- moved D3 15.2 mm to (219.7, 148.6)
- moved R17 15.2 mm to (229.9, 148.6)
- moved R7 15.2 mm to (234.9, 148.6)
- moved Q14 15.2 mm to (235.1, 115.5)
- moved Q4 15.2 mm to (236.2, 119.4)
- moved Q7 15.2 mm to (234.9, 139.7)
- moved R16 15.2 mm to (254.0, 139.7)
- moved R6 15.2 mm to (248.9, 139.7)
- moved D13 15.2 mm to (218.4, 146.0)
- moved Q17 15.2 mm to (236.1, 135.9)
Connections:
- Q13 pad 1: Net-(Q13-S) -> GNDREF
- Q14 pad 3: Net-(Q13-S) -> Net-(Q13-D)
- Q3 pad 1: Net-(Q13-S) -> GNDREF
- Q4 pad 3: Net-(Q13-S) -> Net-(Q13-D)
Routing:
- net GNDREF: track 52.2 -> 108.4 mm, vias 3 -> 4
- net Net-(Q13-D): track 137.4 -> 184.5 mm
- net (no net): track 38.9 -> 64.4 mm
- net VDD: track 478.7 -> 502.2 mm
- net Net-(Q13-S): track 19.6 -> 0.00 mm
- net Net-(Q12-D): track 91.2 -> 106.4 mm, vias 0 -> 2
Other:
- board size 94 x 94 mm -> 94 x 110.5 mm
- board text added: "&"
- board text added: "( A & B ) == !( !A | !B )"
- board text added: "( A | B ) == !( !A & !B )"
- board text added: "(N)AND"
- board text added: "A | B"
- board text added: "NOR"
- board text added: "~{&}"
- board text removed: "(N)OR"
- board text removed: "A & B"
- board text removed: "By putting capacitors around the board, we can ensure that clean power is always available where it will be required."
- board text removed: "In normal use of these demo boards, the capacitors will serve no useful function, and may be omitted!"
- board text removed: "NAND"
- board text removed: "These {dblquote}batteries{dblquote} will help keep local power steady when other logic is causing power fluctuations. You could say it {dblquote}filters noise from the power{dblquote}."
- board text removed: "Transistors require power to {dblquote}switch{dblquote}. One feature of a capacitor is to act like a tiny rechargeable battery."
